Commit message: Use velodyne_description package for 3D lidar simulation

File: otter_gazebo/urdf/otter_gazebo.urdf.xacro (robot description, xacro)
@@ -6,5 +6,5 @@
   <xacro:arg name="imu_enabled"           default="false" />
   <xacro:arg name="lidar_enabled"         default="false" />
-  <xacro:arg name="3d_lidar_enabled"      default="false" />
+  <xacro:arg name="velodyne_enabled"      default="false" />
   <xacro:arg name="top_camera_enabled"    default="false" />
   <xacro:arg name="ground_truth_enabled"  default="false" />
@@ -22,5 +22,5 @@
   <xacro:include filename="$(find otter_gazebo)/urdf/sensors/otter_imu.xacro" />
   <xacro:include filename="$(find otter_gazebo)/urdf/sensors/otter_lidar.xacro" />
-  <xacro:include filename="$(find otter_gazebo)/urdf/sensors/otter_3d_lidar.xacro" />
+  <xacro:include filename="$(find velodyne_description)/urdf/VLP-16.urdf.xacro"/>
   <xacro:include filename="$(find otter_gazebo)/urdf/sensors/otter_camera.xacro" />
   <xacro:include filename="$(find otter_gazebo)/urdf/sensors/otter_p3d.xacro" />
@@ -47,6 +47,8 @@
   </xacro:if>
   <!-- Add 3D LIDAR -->
-  <xacro:if value="$(arg 3d_lidar_enabled)">
-    <xacro:otter_3d_lidar name="3d_lidar" x="-0.2" y="0.0" z="0.6" />
+  <xacro:if value="$(arg velodyne_enabled)">
+    <xacro:VLP-16 parent="base_link" name="velodyne" topic="/velodyne_points" organize_cloud="false" hz="5" samples="440" gpu="false">
+      <origin xyz="-0.2 0.0 0.6" rpy="0 0 0" />
+    </xacro:VLP-16>
   </xacro:if>
   <!-- Add planar LIDAR -->
